Commit message: oops forgot to add params to main file

File: src/cse468_final_bot/urdf/robot.xacro (robot description, xacro)
@@ -5,5 +5,5 @@
         <visual>
             <geometry>
-                <box size="0.8 0.7 0.1"/>
+                <box size="${drivebase_length} ${drivebase_width} ${drivebase_height}"/>
             </geometry>
             <material name="blue"/>

Commit message: fiddiling with nums

File: src/cse468_final_bot/urdf/robot.xacro (robot description, xacro)
@@ -15,5 +15,5 @@
         </collision>
         <inertial>
-            <mass value="25"/>
+            <mass value="55"/>
             <inertia ixx="1.35416" ixy="0.0" ixz="0.0" iyy="2.35416" iyz="0.0" izz="1.04166"/>
         </inertial>
