Commit message: added laser to gazebo

File: src/cse468_final_bot/urdf/laser.xacro (robot description, xacro)
@@ -3,5 +3,5 @@
     <joint name="laser_joint" type="fixed">
         <axis xyz="0.0 1.0 0.0"/>
-        <origin xyz="0 0 ${drivebase_height}" rpy="0.0 0.0 0.0"/>
+        <origin xyz="${drivebase_length/2} 0 ${drivebase_height+0.1}" rpy="0.0 0.0 0.0"/>
         <parent link="base_link"/>
         <child link="hokuyo_link"/>
@@ -27,3 +27,38 @@
         </inertial>
     </link>
+    <gazebo reference="hokuyo_link">
+        <sensor type="ray" name="head_hokuyo_sensor">
+            <pose>0 0 0 0 0 0</pose>
+            <visualize>false</visualize>
+            <update_rate>40</update_rate>
+            <ray>
+                <scan>
+                <horizontal>
+                    <samples>720</samples>
+                    <resolution>1</resolution>
+                    <min_angle>-1.570796</min_angle>
+                    <max_angle>1.570796</max_angle>
+                </horizontal>
+                </scan>
+                <range>
+                <min>0.10</min>
+                <max>30.0</max>
+                <resolution>0.01</resolution>
+                </range>
+                <noise>
+                <type>gaussian</type>
+                <!-- Noise parameters based on published spec for Hokuyo laser
+                    achieving "+-30mm" accuracy at range < 10m.  A mean of 0.0m and
+                    stddev of 0.01m will put 99.7% of samples within 0.03m of the true
+                    reading. -->
+                <mean>0.0</mean>
+                <stddev>0.01</stddev>
+                </noise>
+            </ray>
+            <plugin name="gazebo_ros_head_hokuyo_controller" filename="libgazebo_ros_laser.so">
+                <topicName>/laser/scan</topicName>
+                <frameName>hokuyo_link</frameName>
+            </plugin>
+        </sensor>
+    </gazebo>
 </robot>
