Commit message: added more parameters to make it readable

File: src/cse468_final_bot/urdf/drivebase_macro.xacro (robot description, xacro)
@@ -6,4 +6,8 @@
     <xacro:property name="wheel_radius" value="0.0762"/>
     <xacro:property name="wheel_thickness" value="0.02"/>
+    <xacro:property name="wheel_height" value="-0.01"/>
+    <xacro:property name="center_wheel_drop" value="0.003175"/>
+    <xacro:property name="wheel_base_seperation" value="0.02"/>
+    <xacro:property name="front_rear_spacing" value="0.05"/>
     <xacro:property name="pi" value="3.1415"/>
     <material name="blue">
@@ -27,11 +31,11 @@
             <child link="${position}_${side}_wheel"/>
             <xacro:if value="${position == 'front'}">
-                <origin xyz="${(drivebase_length / 2) + .01} ${((drivebase_width / 2) + .01) * reflect} -0.01"/>
+                <origin xyz="${(drivebase_length / 2) - front_rear_spacing} ${((drivebase_width / 2) + wheel_base_seperation) * reflect} ${wheel_height}"/>
             </xacro:if>
             <xacro:if value="${position == 'center'}">
-                <origin xyz="0 ${((drivebase_width / 2) + .01) * reflect} -0.013175"/>
+                <origin xyz="0 ${((drivebase_width / 2) + wheel_base_seperation) * reflect} ${wheel_height - center_wheel_drop}"/>
             </xacro:if>
             <xacro:if value="${position == 'rear'}">
-                <origin xyz="${-1 * ((drivebase_length / 2) + .01)} ${((drivebase_width / 2) + .01) * reflect} -0.01"/>
+                <origin xyz="${-1 * ((drivebase_length / 2) - front_rear_spacing)} ${((drivebase_width / 2) + wheel_base_seperation) * reflect} ${wheel_height}"/>
             </xacro:if>
             <axis xyz="0 1 0"/>

Commit message: added physics props and tweaked values

File: src/cse468_final_bot/urdf/drivebase_macro.xacro (robot description, xacro)
@@ -5,8 +5,8 @@
     <xacro:property name="drivebase_height" value="0.1"/>
     <xacro:property name="wheel_radius" value="0.0762"/>
-    <xacro:property name="wheel_thickness" value="0.02"/>
+    <xacro:property name="wheel_thickness" value="0.0508"/>
     <xacro:property name="wheel_height" value="-0.01"/>
     <xacro:property name="center_wheel_drop" value="0.003175"/>
-    <xacro:property name="wheel_base_seperation" value="0.02"/>
+    <xacro:property name="wheel_base_seperation" value="0.03"/>
     <xacro:property name="front_rear_spacing" value="0.05"/>
     <xacro:property name="pi" value="3.1415"/>
@@ -26,4 +26,14 @@
                 <material name="white"/>
             </visual>
+            <collision>
+                <geometry>
+                    <cylinder length="${wheel_thickness}" radius="${wheel_radius}"/>
+                </geometry>
+                <origin rpy="0 ${pi / 2} ${pi / 2}" xyz="0 0 0"/>
+            </collision>
+            <inertial>
+                <mass value="0.2630836"/>
+                <inertia ixx="0.000438" ixy="0.0" ixz="0.0" iyy="0.000438" iyz="0.0" izz="0.000763"/>
+            </inertial>
         </link>
         <joint name="base_to_${position}_${side}_wheel" type="continuous">

File: src/cse468_final_bot/urdf/robot.xacro (robot description, xacro)
@@ -9,4 +9,13 @@
             <material name="blue"/>
         </visual>
+        <collision>
+            <geometry>
+                <box size="${drivebase_length} ${drivebase_width} ${drivebase_height}"/>
+            </geometry>
+        </collision>
+        <inertial>
+            <mass value="25"/>
+            <inertia ixx="1.35416" ixy="0.0" ixz="0.0" iyy="2.35416" iyz="0.0" izz="1.04166"/>
+        </inertial>
     </link>
     <xacro:robot_side side="left" reflect="1"/>

Commit message: got basic manual drivebase working

File: src/cse468_final_bot/urdf/drivebase_macro.xacro (robot description, xacro)
@@ -10,5 +10,4 @@
     <xacro:property name="wheel_base_seperation" value="0.03"/>
     <xacro:property name="front_rear_spacing" value="0.05"/>
-    <xacro:property name="pi" value="3.1415"/>
     <material name="blue">
         <color rgba="0 0 0.8 1"/>
@@ -51,4 +50,20 @@
             <axis xyz="0 1 0"/>
         </joint>
+        <transmission name="${position}_${side}_wheel_trans">
+            <type>transmission_interface/SimpleTransmission</type>
+            <actuator name="${position}_${side}_wheel_motor">
+                <mechanicalReduction>7.44</mechanicalReduction>
+            </actuator>
+            <joint name="base_to_${position}_${side}_wheel">
+                <hardwareInterface>VelocityJointInterface</hardwareInterface>
+            </joint>
+        </transmission>
+        <gazebo reference="${position}_${side}_wheel">
+            <mu1 value="200.0"/>
+            <mu2 value="100.0"/>
+            <kp value="10000000.0" />
+            <kd value="1.0" />
+        <material>Gazebo/Grey</material>
+    </gazebo>
     </xacro:macro>
     <xacro:macro name="robot_side" params="side reflect">

File: src/cse468_final_bot/urdf/robot.xacro (robot description, xacro)
@@ -21,3 +21,11 @@
     <xacro:robot_side side="left" reflect="1"/>
     <xacro:robot_side side="right" reflect="-1"/>
+    <gazebo>
+        <static>false</static>
+        <plugin name="gazebo_ros_control" filename="libgazebo_ros_control.so">
+            <robotNamespace>/</robotNamespace>
+            <robotSimType>gazebo_ros_control/DefaultRobotHWSim</robotSimType>
+            <legacyModeNS>true</legacyModeNS>
+        </plugin>
+    </gazebo>
 </robot>

Commit message: added world file

File: src/cse468_final_bot/urdf/drivebase_macro.xacro (robot description, xacro)
@@ -22,5 +22,5 @@
                     <cylinder length="${wheel_thickness}" radius="${wheel_radius}"/>
                 </geometry>
-                <origin rpy="0 ${pi / 2} ${pi / 2}" xyz="0 0 0"/>
+                <origin rpy="0 0 0" xyz="0 0 0"/>
                 <material name="white"/>
             </visual>
@@ -29,5 +29,5 @@
                     <cylinder length="${wheel_thickness}" radius="${wheel_radius}"/>
                 </geometry>
-                <origin rpy="0 ${pi / 2} ${pi / 2}" xyz="0 0 0"/>
+                <origin rpy="0 0 0" xyz="0 0 0"/>
             </collision>
             <inertial>
@@ -40,13 +40,13 @@
             <child link="${position}_${side}_wheel"/>
             <xacro:if value="${position == 'front'}">
-                <origin xyz="${(drivebase_length / 2) - front_rear_spacing} ${((drivebase_width / 2) + wheel_base_seperation) * reflect} ${wheel_height}"/>
+                <origin rpy="${pi / 2} ${pi / 2} 0" xyz="${(drivebase_length / 2) - front_rear_spacing} ${((drivebase_width / 2) + wheel_base_seperation) * reflect} ${wheel_height}"/>
             </xacro:if>
             <xacro:if value="${position == 'center'}">
-                <origin xyz="0 ${((drivebase_width / 2) + wheel_base_seperation) * reflect} ${wheel_height - center_wheel_drop}"/>
+                <origin rpy="${pi / 2} ${pi / 2} 0" xyz="0 ${((drivebase_width / 2) + wheel_base_seperation) * reflect} ${wheel_height - center_wheel_drop}"/>
             </xacro:if>
             <xacro:if value="${position == 'rear'}">
-                <origin xyz="${-1 * ((drivebase_length / 2) - front_rear_spacing)} ${((drivebase_width / 2) + wheel_base_seperation) * reflect} ${wheel_height}"/>
+                <origin rpy="${pi / 2} ${pi / 2} 0" xyz="${-1 * ((drivebase_length / 2) - front_rear_spacing)} ${((drivebase_width / 2) + wheel_base_seperation) * reflect} ${wheel_height}"/>
             </xacro:if>
-            <axis xyz="0 1 0"/>
+            <axis xyz="0 0 1"/>
         </joint>
         <transmission name="${position}_${side}_wheel_trans">
@@ -56,5 +56,5 @@
             </actuator>
             <joint name="base_to_${position}_${side}_wheel">
-                <hardwareInterface>VelocityJointInterface</hardwareInterface>
+                <hardwareInterface>hardware_interface/VelocityJointInterface</hardwareInterface>
             </joint>
         </transmission>

Commit message: trying to get sensor added

File: src/cse468_final_bot/urdf/drivebase_macro.xacro (robot description, xacro)
@@ -64,6 +64,6 @@
             <kp value="10000000.0" />
             <kd value="1.0" />
-        <material>Gazebo/Grey</material>
-    </gazebo>
+            <material>Gazebo/Grey</material>
+        </gazebo>
     </xacro:macro>
     <xacro:macro name="robot_side" params="side reflect">

File: src/cse468_final_bot/urdf/robot.xacro (robot description, xacro)
@@ -2,5 +2,4 @@
 <robot name="robot_with_arm" xmlns:xacro="http://ros.org/wiki/xacro">
     <xacro:include filename="$(find cse468_final_bot)/urdf/drivebase_macro.xacro"/>
-    <xacro:include filename="$(find cse468_final_bot)/urdf/arm_macro.xacro"/>
     <link name="base_link">
         <visual>
@@ -22,4 +21,7 @@
     <xacro:robot_side side="left" reflect="1"/>
     <xacro:robot_side side="right" reflect="-1"/>
+    <!--<xacro:include filename="$(find cse468_final_bot)/urdf/arm_macro.xacro"/>-->
+    <xacro:include filename="$(find cse468_final_bot)/urdf/laser.xacro"/>
+    <xacro:include filename="$(find cse468_final_bot)/urdf/kinect.xacro"/>
     <gazebo>
         <static>false</static>

Commit message: fixed weird drivebase issue

File: src/cse468_final_bot/urdf/drivebase_macro.xacro (robot description, xacro)
@@ -1,13 +1,18 @@
 <?xml version="1.0"?>
-<robot name="drivebase_macros" xmlns:xacro="http://ros.org/wiki/xacro">
-    <xacro:property name="drivebase_length" value="0.8"/>
-    <xacro:property name="drivebase_width" value="0.7"/>
-    <xacro:property name="drivebase_height" value="0.1"/>
-    <xacro:property name="wheel_radius" value="0.0762"/>
-    <xacro:property name="wheel_thickness" value="0.0508"/>
-    <xacro:property name="wheel_height" value="-0.01"/>
-    <xacro:property name="center_wheel_drop" value="0.003175"/>
-    <xacro:property name="wheel_base_seperation" value="0.03"/>
-    <xacro:property name="front_rear_spacing" value="0.05"/>
+<root xmlns:xacro="http://ros.org/wiki/xacro">
+    <xacro:include filename="$(find cse468_final_bot)/urdf/inertia.xacro" />
+    <xacro:property name="front" value="1" />
+    <xacro:property name="middle" value="0" />
+    <xacro:property name="rear" value="-1" />
+    <xacro:property name="left" value="1" />
+    <xacro:property name="right" value="-1" />
+    <xacro:property name="no_drop" value="0" />
+    <xacro:property name="drop" value="-1" />
+    <xacro:property name="high_friction" value="200.0" />
+    <xacro:property name="medium_friction" value="100.0" />
+    <xacro:property name="low_friction" value="1.0" />
+    <xacro:property name="pivot_radius" value="0.025" />
+    <xacro:property name="pivot_height" value="0.025" />
+    <xacro:property name="pivot_mass" value="1.0" />
     <material name="blue">
         <color rgba="0 0 0.8 1"/>
@@ -16,59 +21,58 @@
         <color rgba="1 1 1 1"/>
     </material>
-    <xacro:macro name="wheel" params="side position reflect">
-        <link name="${position}_${side}_wheel">
-            <visual>
-                <geometry>
-                    <cylinder length="${wheel_thickness}" radius="${wheel_radius}"/>
-                </geometry>
-                <origin rpy="0 0 0" xyz="0 0 0"/>
-                <material name="white"/>
-            </visual>
-            <collision>
-                <geometry>
-                    <cylinder length="${wheel_thickness}" radius="${wheel_radius}"/>
-                </geometry>
-                <origin rpy="0 0 0" xyz="0 0 0"/>
-            </collision>
-            <inertial>
-                <mass value="0.2630836"/>
-                <inertia ixx="0.000438" ixy="0.0" ixz="0.0" iyy="0.000438" iyz="0.0" izz="0.000763"/>
-            </inertial>
-        </link>
-        <joint name="base_to_${position}_${side}_wheel" type="continuous">
-            <parent link="base_link"/>
-            <child link="${position}_${side}_wheel"/>
-            <xacro:if value="${position == 'front'}">
-                <origin rpy="${pi / 2} ${pi / 2} 0" xyz="${(drivebase_length / 2) - front_rear_spacing} ${((drivebase_width / 2) + wheel_base_seperation) * reflect} ${wheel_height}"/>
-            </xacro:if>
-            <xacro:if value="${position == 'center'}">
-                <origin rpy="${pi / 2} ${pi / 2} 0" xyz="0 ${((drivebase_width / 2) + wheel_base_seperation) * reflect} ${wheel_height - center_wheel_drop}"/>
-            </xacro:if>
-            <xacro:if value="${position == 'rear'}">
-                <origin rpy="${pi / 2} ${pi / 2} 0" xyz="${-1 * ((drivebase_length / 2) - front_rear_spacing)} ${((drivebase_width / 2) + wheel_base_seperation) * reflect} ${wheel_height}"/>
-            </xacro:if>
-            <axis xyz="0 0 1"/>
-        </joint>
-        <transmission name="${position}_${side}_wheel_trans">
-            <type>transmission_interface/SimpleTransmission</type>
-            <actuator name="${position}_${side}_wheel_motor">
-                <mechanicalReduction>7.44</mechanicalReduction>
-            </actuator>
-            <joint name="base_to_${position}_${side}_wheel">
-                <hardwareInterface>hardware_interface/VelocityJointInterface</hardwareInterface>
+    <xacro:macro name="six_wheel_diff_drive" params="name parent z_offset drop_wheel_height wheel_separation wheelbase_length wheel_radius wheel_width wheel_mass">
+        <xacro:macro name="diff_wheel" params=" parent2 prefix side fntctrbck drop friction mimic mimic_parent">
+            <link name="${prefix}_diff_wheel">
+                <visual>
+                    <geometry>
+                        <cylinder length="${wheel_width}" radius="${wheel_radius}"/>
+                    </geometry>
+                    <origin xyz="0 0 0"/>
+                    <material name="blue"/>
+                </visual>
+                <collision>
+                    <geometry>
+                        <cylinder length="${wheel_width}" radius="${wheel_radius}"/>
+                    </geometry>
+                    <origin xyz="0 0 0"/>
+                </collision>
+                <inertial>
+                    <mass value="${wheel_mass}"/>
+                    <xacro:cylinder_inertia m="${wheel_mass}" r="${wheel_radius}" h="${wheel_width}"/>
+                    <origin xyz="0 0 0"/>
+                </inertial>
+            </link>
+            <joint name="${parent2}_to_${prefix}_diff_wheel" type="continuous">
+                <parent link="${parent2}"/>
+                <child link="${prefix}_diff_wheel"/>
+                <axis xyz="0 0 ${-1*side}"/>
+                <origin rpy="${side*pi/2} 0 0" xyz="${fntctrbck*(wheelbase_length/2)} ${side*(wheel_separation/2)} ${z_offset+drop*drop_wheel_height}"/>
+                <xacro:if value="${mimic != 'NONE'}">
+                    <mimic joint="${mimic_parent}_to_${mimic}_diff_wheel"/>
+                </xacro:if>
             </joint>
-        </transmission>
-        <gazebo reference="${position}_${side}_wheel">
-            <mu1 value="200.0"/>
-            <mu2 value="100.0"/>
-            <kp value="10000000.0" />
-            <kd value="1.0" />
-            <material>Gazebo/Grey</material>
-        </gazebo>
+            <transmission name="${prefix}_diff_wheel_trans">
+                <type>transmission_interface/SimpleTransmission</type>
+                <actuator name="${prefix}_diff_wheel_motor">
+                    <mechanicalReduction>1</mechanicalReduction>
+                </actuator>
+                <joint name="${parent2}_to_${prefix}_diff_wheel">
+                    <hardwareInterface>hardware_interface/VelocityJointInterface</hardwareInterface>
+                </joint>
+            </transmission>
+            <gazebo reference="${prefix}_diff_wheel">
+                <mu1 value="${friction}"/>
+                <mu2 value="${friction}"/>
+                <kp value="10000000.0"/>
+                <kd value="1.0" />
+                <material>Gazebo/gray</material>
+            </gazebo>
+        </xacro:macro>
+        <xacro:diff_wheel parent2="${parent}" prefix="fl" side="${left}" fntctrbck="${front}" drop="${no_drop}" friction="${low_friction}" mimic="ml" mimic_parent="base_link"/>
+        <xacro:diff_wheel parent2="${parent}" prefix="ml" side="${left}" fntctrbck="${middle}" drop="${drop}" friction="${high_friction}" mimic="NONE" mimic_parent="base_link"/>
+        <xacro:diff_wheel parent2="${parent}" prefix="rl" side="${left}" fntctrbck="${rear}" drop="${no_drop}" friction="${low_friction}"  mimic="ml" mimic_parent="base_link"/>
+        <xacro:diff_wheel parent2="${parent}" prefix="fr" side="${right}" fntctrbck="${front}" drop="${no_drop}" friction="${low_friction}"  mimic="mr" mimic_parent="base_link"/>
+        <xacro:diff_wheel parent2="${parent}" prefix="mr" side="${right}" fntctrbck="${middle}" drop="${drop}" friction="${high_friction}"  mimic="NONE" mimic_parent="base_link"/>
+        <xacro:diff_wheel parent2="${parent}" prefix="rr" side="${right}" fntctrbck="${rear}" drop="${no_drop}" friction="${low_friction}"  mimic="mr" mimic_parent="base_link"/>
     </xacro:macro>
-    <xacro:macro name="robot_side" params="side reflect">
-        <xacro:wheel side="${side}" position="front" reflect="${reflect}"/>
-        <xacro:wheel side="${side}" position="center" reflect="${reflect}"/>
-        <xacro:wheel side="${side}" position="rear" reflect="${reflect}"/>
-    </xacro:macro>
-</robot>
+</root>

File: src/cse468_final_bot/urdf/kinect.xacro (robot description, xacro)
@@ -22,5 +22,5 @@
     <joint name="camera_joint" type="fixed">
         <axis xyz="0.0 0.0 0.0"/>
-        <origin xyz="${drivebase_length/2} 0 ${drivebase_height + .01}" rpy="0.0 0.0 0.0"/>
+        <origin xyz=".35 0 0.2" rpy="0.0 0.0 0.0"/>
         <parent link="base_link"/>
         <child link="camera_link"/>
@@ -48,9 +48,9 @@
                 <updateRate>0.0</updateRate>
                 <cameraName>camera_ir</cameraName>
-                <imageTopicName>/camera/color/image_raw</imageTopicName>
-                <cameraInfoTopicName>/camera/color/camera_info</cameraInfoTopicName>
-                <depthImageTopicName>/camera/depth/image_raw</depthImageTopicName>
-                <depthImageCameraInfoTopicName>/camera/depth/camera_info</depthImageCameraInfoTopicName>
-                <pointCloudTopicName>/camera/depth/points</pointCloudTopicName>
+                <imageTopicName>color/image_raw</imageTopicName>
+                <cameraInfoTopicName>color/camera_info</cameraInfoTopicName>
+                <depthImageTopicName>depth/image_raw</depthImageTopicName>
+                <depthImageCameraInfoTopicName>depth/camera_info</depthImageCameraInfoTopicName>
+                <pointCloudTopicName>depth/points</pointCloudTopicName>
                 <frameName>camera_link</frameName>
                 <pointCloudCutoff>0.5</pointCloudCutoff>

File: src/cse468_final_bot/urdf/laser.xacro (robot description, xacro)
@@ -3,5 +3,5 @@
     <joint name="laser_joint" type="fixed">
         <axis xyz="0.0 1.0 0.0"/>
-        <origin xyz="${drivebase_length/2} 0 ${drivebase_height+0.1}" rpy="0.0 0.0 0.0"/>
+        <origin xyz=".35 0 0.4" rpy="0.0 0.0 0.0"/>
         <parent link="base_link"/>
         <child link="hokuyo_link"/>

File: src/cse468_final_bot/urdf/robot.xacro (robot description, xacro)
@@ -2,23 +2,8 @@
 <robot name="robot_with_arm" xmlns:xacro="http://ros.org/wiki/xacro">
     <xacro:include filename="$(find cse468_final_bot)/urdf/drivebase_macro.xacro"/>
-    <link name="base_link">
-        <visual>
-            <geometry>
-                <box size="${drivebase_length} ${drivebase_width} ${drivebase_height}"/>
-            </geometry>
-            <material name="blue"/>
-        </visual>
-        <collision>
-            <geometry>
-                <box size="${drivebase_length} ${drivebase_width} ${drivebase_height}"/>
-            </geometry>
-        </collision>
-        <inertial>
-            <mass value="55"/>
-            <inertia ixx="1.35416" ixy="0.0" ixz="0.0" iyy="2.35416" iyz="0.0" izz="1.04166"/>
-        </inertial>
-    </link>
-    <xacro:robot_side side="left" reflect="1"/>
-    <xacro:robot_side side="right" reflect="-1"/>
+    <xacro:include filename="$(find cse468_final_bot)/urdf/chassis.xacro" />
+    <link name="base_link"/>
+    <xacro:robot_chassis name="chassis" parent="base_link" z_offset="0.0" chassis_length="0.8128" chassis_width="0.7112" chassis_height="0.1524" chassis_mass="50"/>
+    <xacro:six_wheel_diff_drive name="tank_drive" parent="base_link" z_offset="0.0" drop_wheel_height="0.003175" wheel_separation="0.6096" wheelbase_length="0.6096" wheel_radius="0.1016" wheel_width="0.0381" wheel_mass="1"/>
     <!--<xacro:include filename="$(find cse468_final_bot)/urdf/arm_macro.xacro"/>-->
     <xacro:include filename="$(find cse468_final_bot)/urdf/laser.xacro"/>
