Commit message: changed pos of kinect

File: src/cse468_final_bot/urdf/kinect.xacro (robot description, xacro)
@@ -3,5 +3,5 @@
     <joint name="camera_joint" type="fixed">
         <axis xyz="0.0 0.0 0.0"/>
-        <origin xyz="${drivebase_length + 0.1} 0 ${drivebase_height + .05}" rpy="0.0 0.0 0.0"/>
+        <origin xyz="${drivebase_length/2} 0 ${drivebase_height + .01}" rpy="0.0 0.0 0.0"/>
         <parent link="base_link"/>
         <child link="camera_link"/>
@@ -21,5 +21,5 @@
         </visual>
         <inertial>
-            <mass value="1e-5" />
+            <mass value="0.05" />
             <origin xyz="0 0 0" rpy="0 0 0"/>
             <inertia ixx="1e-6" ixy="0" ixz="0" iyy="1e-6" iyz="0" izz="1e-6" />

File: src/cse468_final_bot/urdf/laser.xacro (robot description, xacro)
@@ -22,5 +22,5 @@
         </visual>
         <inertial>
-            <mass value="1e-5" />
+            <mass value="0.05" />
             <origin xyz="0 0 0" rpy="0 0 0"/>
             <inertia ixx="1e-6" ixy="0" ixz="0" iyy="1e-6" iyz="0" izz="1e-6" />

Commit message: changed back to empty world

File: src/cse468_final_bot/urdf/kinect.xacro (robot description, xacro)
@@ -1,10 +1,4 @@
 <?xml version="1.0"?>
 <robot name="kinect" xmlns:xacro="http://ros.org/wiki/xacro">
-    <joint name="camera_joint" type="fixed">
-        <axis xyz="0.0 0.0 0.0"/>
-        <origin xyz="${drivebase_length/2} 0 ${drivebase_height + .01}" rpy="0.0 0.0 0.0"/>
-        <parent link="base_link"/>
-        <child link="camera_link"/>
-    </joint>
     <link name="camera_link">
         <collision>
@@ -26,3 +20,52 @@
         </inertial>
     </link>
+    <joint name="camera_joint" type="fixed">
+        <axis xyz="0.0 0.0 0.0"/>
+        <origin xyz="${drivebase_length/2} 0 ${drivebase_height + .01}" rpy="0.0 0.0 0.0"/>
+        <parent link="base_link"/>
+        <child link="camera_link"/>
+    </joint>
+    <gazebo reference="camera_link">
+        <sensor type="depth" name="camera1">
+            <update_rate>30.0</update_rate>
+            <camera name="head">
+                <horizontal_fov>1.3962634</horizontal_fov>
+                <image>
+                <width>800</width>
+                <height>800</height>
+                <format>R8G8B8</format>
+                </image>
+                <clip>
+                <near>0.02</near>
+                <far>300</far>
+                </clip>
+            </camera>
+            <plugin name="camera_plugin" filename="libgazebo_ros_openni_kinect.so">
+                <baseline>0.2</baseline>
+                <alwaysOn>true</alwaysOn>
+                <!-- Keep this zero, update_rate in the parent <sensor> tag
+                    will control the frame rate. -->
+                <updateRate>0.0</updateRate>
+                <cameraName>camera_ir</cameraName>
+                <imageTopicName>/camera/color/image_raw</imageTopicName>
+                <cameraInfoTopicName>/camera/color/camera_info</cameraInfoTopicName>
+                <depthImageTopicName>/camera/depth/image_raw</depthImageTopicName>
+                <depthImageCameraInfoTopicName>/camera/depth/camera_info</depthImageCameraInfoTopicName>
+                <pointCloudTopicName>/camera/depth/points</pointCloudTopicName>
+                <frameName>camera_link</frameName>
+                <pointCloudCutoff>0.5</pointCloudCutoff>
+                <pointCloudCutoffMax>3.0</pointCloudCutoffMax>
+                <distortionK1>0</distortionK1>
+                <distortionK2>0</distortionK2>
+                <distortionK3>0</distortionK3>
+                <distortionT1>0</distortionT1>
+                <distortionT2>0</distortionT2>
+                <CxPrime>0</CxPrime>
+                <Cx>0</Cx>
+                <Cy>0</Cy>
+                <focalLength>0</focalLength>
+                <hackBaseline>0</hackBaseline>
+            </plugin>
+        </sensor>
+    </gazebo>
 </robot>

Commit message: refining slam need to add motor to arm

File: src/cse468_final_bot/urdf/kinect.xacro (robot description, xacro)
@@ -22,5 +22,5 @@
     <joint name="camera_joint" type="fixed">
         <axis xyz="0.0 0.0 0.0"/>
-        <origin xyz=".35 0 0.2" rpy="0.0 0.0 0.0"/>
+        <origin xyz=".35 0 0.4" rpy="0.0 0.0 0.0"/>
         <parent link="base_link"/>
         <child link="camera_link"/>

File: src/cse468_final_bot/urdf/laser.xacro (robot description, xacro)
@@ -3,5 +3,5 @@
     <joint name="laser_joint" type="fixed">
         <axis xyz="0.0 1.0 0.0"/>
-        <origin xyz=".35 0 0.4" rpy="0.0 0.0 0.0"/>
+        <origin xyz=".35 0 0.2" rpy="0.0 0.0 0.0"/>
         <parent link="base_link"/>
         <child link="hokuyo_link"/>
