Commit message: arm moves now and also connects to drivebase

File: src/cse468_final_bot/urdf/arm_macro.xacro (robot description, xacro)
@@ -1,43 +1,116 @@
 <?xml version="1.0"?>
-<robot name="arm_macros"
-    xmlns:xacro="http://ros.org/wiki/xacro">
+<!-- Revolute-Revolute Manipulator -->
+<robot
+    xmlns:xacro="http://www.ros.org/wiki/xacro" name="rrbot">
+    <!--<xacro:include filename="$(find cse468_final_bot)/urdf/gripper.xacro" />-->
+    <!-- Constants for robot dimensions -->
+    <xacro:property name="width" value="0.1" />
+    <xacro:property name="height1" value="1" />
+    <xacro:property name="height2" value=".5" />
+    <xacro:property name="height3" value=".5" />
+    <xacro:property name="axle_offset" value="0.05" />
+    <xacro:property name="damp" value="0.7" />
+    <!-- Base Link -->
     <joint name="gripper_extension" type="fixed">
         <parent link="base_link"/>
-        <child link="vert"/>
-        <origin rpy="0 0 0" xyz="0.19 0 0.2"/>
+        <child link="base_link2"/>
+        <origin rpy="0 0 0" xyz="0 0 0"/>
     </joint>
-    <link name="vert">
+    <link name="base_link2">
         <visual>
+            <origin xyz="0 0 ${height1/2}" rpy="0 0 0" />
             <geometry>
-                <cylinder length="0.4" radius="0.02"/>
+                <box size="${width} ${width} ${height1}" />
             </geometry>
-            <origin rpy="0 0 0 " xyz="-0.2 0 0"/>
         </visual>
+        <collision>
+            <origin xyz="0 0 ${height1/2}" rpy="0 0 0" />
+            <geometry>
+                <box size="${width} ${width} ${height1}" />
+            </geometry>
+        </collision>
+        <inertial>
+            <origin xyz="0 0 ${height1/2}" rpy="0 0 0" />
+            <mass value="1" />
+            <inertia ixx="1.0" ixy="0.0" ixz="0.0" iyy="1.0" iyz="0.0" izz="1.0" />
+        </inertial>
     </link>
-    <joint name="init_joint" type="fixed">
-        <origin rpy="0 0 0" xyz="0.2 0.01 0"/>
-        <parent link="vert"/>
-        <child link="gripper_pole"/>
+    <!-- Joint between Base Link and Middle Link -->
+    <joint name="joint_base_mid" type="revolute">
+        <parent link="base_link2" />
+        <child link="mid_link" />
+        <origin xyz="0 ${width} ${height1 - axle_offset}" rpy="0 0  0" />
+        <axis xyz="0 1 0" />
+        <dynamics damping="${damp}" />
+        <limit effort="100.0" velocity="0.5" lower="-3.14" upper="3.14" />
     </joint>
-    <link name="gripper_pole">
+    <!-- Middle Link -->
+    <link name="mid_link">
         <visual>
+            <origin xyz="0 0 ${height2/2 - axle_offset}" rpy="0 0 0" />
             <geometry>
-                <cylinder length="0.4" radius="0.02"/>
+                <box size="${width} ${width} ${height2}" />
             </geometry>
-            <origin rpy="0 1.57075 0 " xyz="0 0 0"/>
         </visual>
+        <collision>
+            <origin xyz="0 0 ${height2/2 - axle_offset}" rpy="0 0 0" />
+            <geometry>
+                <box size="${width} ${width} ${height2}" />
+            </geometry>
+        </collision>
+        <inertial>
+            <origin xyz="0 0 ${height2/2 - axle_offset}" rpy="0 0 0" />
+            <mass value="1" />
+            <inertia ixx="1.0" ixy="0.0" ixz="0.0" iyy="1.0" iyz="0.0" izz="1.0" />
+        </inertial>
     </link>
-    <joint name="left_gripper_joint" type="fixed">
-        <origin rpy="0 0 0" xyz="0.2 0.01 0"/>
-        <parent link="gripper_pole"/>
+    <!-- Joint between Middle Link and Top Link -->
+    <joint name="joint_mid_top" type="revolute">
+        <parent link="mid_link" />
+        <child link="top_link" />
+        <origin xyz="0 ${width} ${height2 - axle_offset*2}" rpy="0 0  0" />
+        <axis xyz="0 1 0" />
+        <dynamics damping="${damp}" />
+        <limit effort="100.0" velocity="0.5" lower="-3.14" upper="3.14" />
+    </joint>
+    <!-- Top Link -->
+    <link name="top_link">
+        <visual>
+            <origin xyz="0 0 ${height3/2 - axle_offset}" rpy="0 0 0" />
+            <geometry>
+                <box size="${width} ${width} ${height3}" />
+            </geometry>
+        </visual>
+        <collision>
+            <origin xyz="0 0 ${height3/2 - axle_offset}" rpy="0 0 0" />
+            <geometry>
+                <box size="${width} ${width} ${height3}" />
+            </geometry>
+        </collision>
+        <inertial>
+            <origin xyz="0 0 ${height3/2 - axle_offset}" rpy="0 0 0" />
+            <mass value="1" />
+            <inertia ixx="1.0" ixy="0.0" ixz="0.0" iyy="1.0" iyz="0.0" izz="1.0" />
+        </inertial>
+    </link>
+    <joint name="left_gripper_joint" type="revolute">
+        <parent link="top_link"/>
         <child link="left_gripper"/>
+        <origin xyz="0 0 ${height2 - axle_offset}" rpy="0 -1.57 0"/>
+        <axis xyz="0 0 1"/>
+        <limit effort="30.0" lower="-0.548" upper="0.0" velocity="0.1"/>
     </joint>
     <link name="left_gripper">
         <visual>
-            <origin rpy="0.0 0 0" xyz="0 0 0"/>
+            <origin rpy="0 0 0" xyz="0 0 0"/>
             <geometry>
                 <mesh filename="package://urdf_tutorial/meshes/l_finger.dae"/>
             </geometry>
         </visual>
+        <collision>
+            <geometry>
+                <box size="0.1 0.1 0.1"/>
+            </geometry>
+        </collision>
     </link>
     <joint name="left_tip_joint" type="fixed">
@@ -47,14 +120,22 @@
     <link name="left_tip">
         <visual>
-            <origin rpy="0.0 0 0" xyz="0.09137 0.00495 0"/>
+            <origin rpy="0 0 0" xyz="0.09137 0.00495 0"/>
             <geometry>
-                <mesh filename="package://urdf_tutorial/meshes/l_finger_tip.dae"/>
+                <mesh
+          filename="package://urdf_tutorial/meshes/l_finger_tip.dae"/>
             </geometry>
         </visual>
+        <collision>
+            <geometry>
+                <box size="0.1 0.1 0.1"/>
+            </geometry>
+        </collision>
     </link>
-    <joint name="right_gripper_joint" type="fixed">
-        <origin rpy="0 0 0" xyz="0.2 -0.01 0"/>
-        <parent link="gripper_pole"/>
+    <joint name="right_gripper_joint" type="revolute">
+        <parent link="top_link"/>
         <child link="right_gripper"/>
+        <origin xyz="0 0 ${height2 - axle_offset}" rpy="0 -1.57 0"/>
+        <axis xyz="0 0 -1"/>
+        <limit effort="30.0" lower="0.0" upper="0.548" velocity="0.5"/>
     </joint>
     <link name="right_gripper">
@@ -65,4 +146,9 @@
             </geometry>
         </visual>
+        <collision>
+            <geometry>
+                <box size="0.1 0.1 0.1"/>
+            </geometry>
+        </collision>
     </link>
     <joint name="right_tip_joint" type="fixed">
@@ -77,4 +163,9 @@
             </geometry>
         </visual>
+        <collision>
+            <geometry>
+                <box size="0.1 0.1 0.1"/>
+            </geometry>
+        </collision>
     </link>
 </robot>

File: src/cse468_final_bot/urdf/robot.xacro (robot description, xacro)
@@ -21,7 +21,7 @@
     <xacro:robot_side side="left" reflect="1"/>
     <xacro:robot_side side="right" reflect="-1"/>
-    <!--<xacro:include filename="$(find cse468_final_bot)/urdf/arm_macro.xacro"/>-->
+    <xacro:include filename="$(find cse468_final_bot)/urdf/arm_macro.xacro"/>
     <xacro:include filename="$(find cse468_final_bot)/urdf/laser.xacro"/>
-    <xacro:include filename="$(find cse468_final_bot)/urdf/kinect.xacro"/>
+   <xacro:include filename="$(find cse468_final_bot)/urdf/kinect.xacro"/>
     <gazebo>
         <static>false</static>

Commit message: added moveit

File: src/cse468_final_bot/urdf/arm_macro.xacro (robot description, xacro)
@@ -169,3 +169,35 @@
         </collision>
     </link>
+    <transmission name="middle_link_trans">
+        <type>transmission_interface/SimpleTransmission</type>
+        <actuator name="middle_link_motor">
+            <mechanicalReduction>1</mechanicalReduction>
+        </actuator>
+        <joint name="joint_base_mid">
+            <hardwareInterface>hardware_interface/PositionJointInterface</hardwareInterface>
+        </joint>
+    </transmission>
+    <gazebo reference="middle_link">
+        <mu1 value="0.01"/>
+        <mu2 value="0.01"/>
+        <kp value="10000000.0"/>
+        <kd value="1.0" />
+        <material>Gazebo/gray</material>
+    </gazebo>
+    <transmission name="top_link_trans">
+        <type>transmission_interface/SimpleTransmission</type>
+        <actuator name="top_link_motor">
+            <mechanicalReduction>1</mechanicalReduction>
+        </actuator>
+        <joint name="joint_mid_top">
+            <hardwareInterface>hardware_interface/PositionJointInterface</hardwareInterface>
+        </joint>
+    </transmission>
+    <gazebo reference="top_link">
+        <mu1 value="0.01"/>
+        <mu2 value="0.01"/>
+        <kp value="10000000.0"/>
+        <kd value="1.0" />
+        <material>Gazebo/gray</material>
+    </gazebo>
 </robot>
